Commit message: Ready for Navigation

File: src/mobile_robot_description/urdf/camera_sensor.xacro (robot description, xacro)
@@ -29,27 +29,24 @@
     <gazebo reference="camera_link">
         <sensor name="camera" type="camera">
-            <camera>
-                <horizontal_fov>1.3962634</horizontal_fov>
-                <image>
-                    <width>640</width>
-                    <height>480</height>
-                    <format>R8G8B8</format>
-                </image>
-                <clip>
-                    <near>0.1</near>
-                    <far>15</far>
-                </clip>
-                <noise>
-                    <type>gaussian</type>
-                    <mean>0.0</mean>
-                    <stddev>0.007</stddev>
-                </noise>
-                <optical_frame_id>camera_link_optical</optical_frame_id>
-                <camera_info_topic>camera/camera_info</camera_info_topic>
-            </camera>
-            <always_on>1</always_on>
-            <update_rate>20</update_rate>
-            <visualize>true</visualize>
-            <topic>camera/image_raw</topic>
+        <pose>0 0 0 0 0 0</pose>
+        <camera>
+            <horizontal_fov>1.047</horizontal_fov>
+            <image>
+            <width>640</width>
+            <height>480</height>
+            <format>RGB_INT8</format>
+            </image>
+            <clip>
+            <near>0.1</near>
+            <far>100</far>
+            </clip>
+        </camera>
+        <always_on>1</always_on>
+        <update_rate>30</update_rate>
+        <visualize>true</visualize>
+        <topic>/camera/image_raw</topic> <!-- Gazebo topic -->
+        <plugin name="gz::sim::systems::Sensors" filename="gz-sim-sensors-system">
+            <render_engine>ogre2</render_engine>
+        </plugin>
         </sensor>
     </gazebo>

File: src/mobile_robot_description/urdf/lidar.xacro (robot description, xacro)
@@ -1,32 +1,58 @@
 <?xml version="1.0"?>
 <robot xmlns:xacro="http://www.ros.org/wiki/xacro">
+    <link name ="lidar_link">
+        <visual>
+            <geometry>
+                <cylinder radius = "${radius}" length = "${length}"/>
+            </geometry>
+            <origin xyz = "0 0 0" rpy = "0 0 0"/>
+            <material name = "white"/>
+        </visual>
+        <collision>
+            <geometry>
+                <cylinder radius = "${radius}" length = "${length}"/>
+            </geometry>
+            <origin xyz = "0 0 0" rpy = "0 0 0"/>
+        </collision>
+        <xacro:wheel m = "1.0" r = "${radius}" h = "${length}"
+                             o_xyz = "0 0 0" o_rpy = "0 0 0"/>
+    </link>
+    <joint name = "base_lidar_joint" type = "fixed">
+        <parent link = "base_link"/>
+        <child link = "lidar_link"/>
+        <origin xyz = "0 0 ${base_height + length / 2.0}" rpy = "0 0 0"/>
+    </joint>
     <gazebo reference="lidar_link">
-        <material>Gazebo/Red</material>
-        <sensor name="lidar_sensor" type="ray">
-            <pose>0 0 0.1 0 0 0</pose>
+        <!-- <material>Gazebo/Red</material> -->
+          <sensor name="lidar" type="gpu_lidar">
+            <always_on>true</always_on>
             <visualize>true</visualize>
-            <update_rate>20</update_rate>
-            <ray>
+            <update_rate>10</update_rate>
+            <topic>/lidar/scan</topic>
+            <gz_frame_id>lidar_link</gz_frame_id>
+            <lidar>
             <scan>
                 <horizontal>
                 <samples>360</samples>
-                <min_angle>-3.14</min_angle>
-                <max_angle>3.14</max_angle>
+                <resolution>1.000000</resolution>
+                <min_angle>-3.14159</min_angle>
+                <max_angle>3.14159</max_angle>
                 </horizontal>
             </scan>
             <range>
-                <min>0.3</min>
-                <max>10.0</max>
+                <min>0.120000</min>
+                <max>10</max>
+                <resolution>0.01</resolution>
             </range>
-            </ray>
-            <plugin name="gazebo_ros_lidar_controller" filename="libgazebo_ros_ray_sensor.so">
-            <ros>
-                <namespace>/</namespace>
-                <remapping>~/out:=scan</remapping>
-            </ros>
-            <output_type>sensor_msgs/LaserScan</output_type>
-            <frame_name>lidar_link</frame_name>
-            </plugin>
+            <noise>
+                <type>gaussian</type>
+                <mean>0.0</mean>
+                <stddev>0.01</stddev>
+            </noise>
+            </lidar>
         </sensor>
+        <plugin filename="gz-sim-sensors-system" name="gz::sim::systems::Sensors">
+            <render_engine>ogre2</render_engine>
+        </plugin>
     </gazebo>
 </robot>

File: src/mobile_robot_description/urdf/mobile_base.xacro (robot description, xacro)
@@ -25,21 +25,4 @@
         <xacro:box_inertia m = "5.0" x = "${base_len}" y = "${base_width}" z = "${base_height}"
                            o_xyz = "0 0 ${radius}" o_rpy = "0 0 0"/>
-    </link>
-    <link name ="lidar_link">
-        <visual>
-            <geometry>
-                <cylinder radius = "${radius}" length = "${length}"/>
-            </geometry>
-            <origin xyz = "0 0 0" rpy = "0 0 0"/>
-            <material name = "white"/>
-        </visual>
-        <!-- <collision>
-            <geometry>
-                <cylinder radius = "${radius}" length = "${length}"/>
-            </geometry>
-            <origin xyz = "0 0 0" rpy = "0 0 0"/>
-        </collision>
-        <xacro:wheel m = "1.0" r = "${radius}" h = "${length}"
-                             o_xyz = "0 0 0" o_rpy = "0 0 0"/> -->
     </link>
     <xacro:macro name = "wheel_link" params="prefix">
@@ -85,10 +68,5 @@
         <origin xyz = "0 0 ${radius}" rpy = "0 0 0"/>
     </joint>
-    <joint name = "base_lidar_joint" type = "fixed">
-        <parent link = "base_link"/>
-        <child link = "lidar_link"/>
-        <origin xyz = "0 0 ${base_height + length / 2.0}" rpy = "0 0 0"/>
-    </joint>
-    <joint name = "base_wheel_joint_1" type = "continuous">
+    <joint name = "left_wheel_joint" type = "continuous">
         <parent link = "base_link"/>
         <child link = "left_wheel_link"/>
@@ -96,5 +74,5 @@
         <axis xyz = "0 1 0"/>
     </joint>
-    <joint name = "base_wheel_joint_2" type = "continuous">
+    <joint name = "right_wheel_joint" type = "continuous">
         <parent link = "base_link"/>
         <child link = "right_wheel_link"/>

File: src/mobile_robot_description/urdf/mobile_base_gazebo.xacro (robot description, xacro)
@@ -1,4 +1,10 @@
 <?xml version="1.0"?>
 <robot xmlns:xacro="http://www.ros.org/wiki/xacro">
+    <gazebo>
+      <plugin filename="gz-sim-joint-state-publisher-system" name="gz::sim::systems::JointStatePublisher">
+          <joint_name>left_wheel_joint</joint_name>
+          <joint_name>right_wheel_joint</joint_name>
+      </plugin>
+  </gazebo>
   <gazebo reference="caster_wheel">
         <mu1 value="0.1"/>
@@ -7,16 +13,13 @@
   <gazebo>
       <plugin filename="gz-sim-diff-drive-system" name="gz::sim::systems::DiffDrive">
-          <left_joint>base_wheel_joint_1</left_joint>
-          <right_joint>base_wheel_joint_2</right_joint>
+          <left_joint>left_wheel_joint</left_joint>
+          <right_joint>right_wheel_joint</right_joint>
           <wheel_separation>0.425</wheel_separation>
           <wheel_radius>0.1</wheel_radius>
+          <topic>/cmd_vel</topic>
           <frame_id>odom</frame_id>
           <child_frame_id>base_footprint</child_frame_id>
-      </plugin>
-  </gazebo>
-  <gazebo>
-      <plugin filename="gz-sim-joint-state-publisher-system" name="gz::sim::systems::JointStatePublisher">
-          <joint_name>base_wheel_joint_1</joint_name>
-          <joint_name>base_wheel_joint_2</joint_name>
+          <publish_tf>true</publish_tf>
+          <odom_topic>/odom</odom_topic>
       </plugin>
   </gazebo>

File: src/mobile_robot_description/urdf/my_car.urdf.xacro (robot description, xacro)
@@ -3,8 +3,6 @@
     <xacro:include filename = "common_properties.xacro"/>
     <xacro:include filename = "mobile_base.xacro"/>
-    <!-- <xacro:include filename = "mobile_base.ros2_control.xacro"/> -->
-    <xacro:include filename = "mobile_base_gazebo.xacro"/>
-    <xacro:include filename = "gazebo_plugin.xacro"/>
     <xacro:include filename = "camera_sensor.xacro"/>
     <xacro:include filename = "lidar.xacro"/>
+    <xacro:include filename = "mobile_base_gazebo.xacro"/>
 </robot>

Commit message: added gazebo world map for autonomous driving

File: src/mobile_robot_description/urdf/camera_sensor.xacro (robot description, xacro)
@@ -1,52 +1,62 @@
 <?xml version="1.0"?>
 <robot xmlns:xacro="http://www.ros.org/wiki/xacro">
-    <xacro:property name = "camera_len" value = "0.01"/>
-    <xacro:property name = "camera_width" value = "0.15"/>
-    <xacro:property name = "camera_height" value = "0.08"/>
-    <link name = "camera_link">
+    <xacro:property name="camera_len" value="0.01"/>
+    <xacro:property name="camera_width" value="0.15"/>
+    <xacro:property name="camera_height" value="0.08"/>
+    <!-- Main camera link (physical box) -->
+    <link name="camera_link">
         <visual>
             <geometry>
-                <box size = "${camera_len} ${camera_width} ${camera_height}"/>
+                <box size="${camera_len} ${camera_width} ${camera_height}"/>
             </geometry>
-            <origin xyz = "0 0 0" rpy = "0 0 0"/>
-            <material name = "white"/>
+            <origin xyz="0 0 0" rpy="0 0 0"/>
+            <material name="white"/>
         </visual>
         <collision>
             <geometry>
-                <box size = "${camera_len} ${camera_width} ${camera_height}"/>
+                <box size="${camera_len} ${camera_width} ${camera_height}"/>
             </geometry>
-            <origin xyz = "0 0 0" rpy = "0 0 0"/>
+            <origin xyz="0 0 0" rpy="0 0 0"/>
         </collision>
-        <xacro:box_inertia m = "0.5" x = "${camera_len}" y = "${camera_width}" z = "${camera_height}"
-                            o_xyz = "0 0 0" o_rpy = "0 0 0"/>
+        <xacro:box_inertia m="0.5" x="${camera_len}" y="${camera_width}" z="${camera_height}"
+                            o_xyz="0 0 0" o_rpy="0 0 0"/>
     </link>
-    <joint name  = "camera_link_joint" type = "fixed">
-        <parent link = "base_link"/>
-        <child link = "camera_link"/>
-        <origin xyz = "${base_len / 2} 0 ${base_height / 2}" rpy = "0 0 0"/>
-        <axis xyz = "0 1 0"/>
+    <!-- Optical frame (for ROS camera convention) -->
+    <link name="camera_link_optical"/>
+    <!-- Joint from camera_link to camera_link_optical -->
+    <joint name="camera_link_optical_joint" type="fixed">
+        <parent link="camera_link"/>
+        <child link="camera_link_optical"/>
+        <!-- Rotate so that optical frame has X right, Y down, Z forward -->
+        <origin xyz="0 0 0" rpy="${-pi/2} 0 ${-pi/2}"/>
     </joint>
-    <gazebo reference="camera_link">
+    <!-- Attach camera_link to base_link -->
+    <joint name="camera_link_joint" type="fixed">
+        <parent link="base_link"/>
+        <child link="camera_link"/>
+        <origin xyz="${base_len / 2} 0 ${base_height / 2}" rpy="0 0 0"/>
+        <axis xyz="0 1 0"/>
+    </joint>
+    <!-- Gazebo camera sensor (Harmonic version) -->
+    <gazebo reference="camera_link">   <!-- Attach sensor to optical link -->
         <sensor name="camera" type="camera">
-        <pose>0 0 0 0 0 0</pose>
-        <camera>
-            <horizontal_fov>1.047</horizontal_fov>
-            <image>
-            <width>640</width>
-            <height>480</height>
-            <format>RGB_INT8</format>
-            </image>
-            <clip>
-            <near>0.1</near>
-            <far>100</far>
-            </clip>
-        </camera>
-        <always_on>1</always_on>
-        <update_rate>30</update_rate>
-        <visualize>true</visualize>
-        <topic>/camera/image_raw</topic> <!-- Gazebo topic -->
-        <plugin name="gz::sim::systems::Sensors" filename="gz-sim-sensors-system">
-            <render_engine>ogre2</render_engine>
-        </plugin>
+            <pose>0 0 0 0 0 0</pose>          <!-- relative to camera_link_optical -->
+            <camera>
+                <horizontal_fov>1.047</horizontal_fov>
+                <image>
+                    <width>640</width>
+                    <height>480</height>
+                    <format>R8G8B8</format>   <!-- Preferred format in Harmonic -->
+                </image>
+                <clip>
+                    <near>0.1</near>
+                    <far>100</far>
+                </clip>
+            </camera>
+            <always_on>1</always_on>
+            <update_rate>30</update_rate>
+            <visualize>true</visualize>
+            <topic>/camera</topic>    <!-- Must match bridge gz_topic_name -->
+            <gz_frame_id>camera_link_optical</gz_frame_id>   <!-- Frame in Gazebo messages -->
         </sensor>
     </gazebo>

File: src/mobile_robot_description/urdf/lidar.xacro (robot description, xacro)
@@ -29,5 +29,5 @@
             <visualize>true</visualize>
             <update_rate>10</update_rate>
-            <topic>/lidar/scan</topic>
+            <topic>/scan</topic>                   <!-- Must be Same as Gazebo bridge topic name-->
             <gz_frame_id>lidar_link</gz_frame_id>
             <lidar>
@@ -42,5 +42,5 @@
             <range>
                 <min>0.120000</min>
-                <max>10</max>
+                <max>10.00</max>
                 <resolution>0.01</resolution>
             </range>
@@ -52,7 +52,4 @@
             </lidar>
         </sensor>
-        <plugin filename="gz-sim-sensors-system" name="gz::sim::systems::Sensors">
-            <render_engine>ogre2</render_engine>
-        </plugin>
     </gazebo>
 </robot>

File: src/mobile_robot_description/urdf/mobile_base_gazebo.xacro (robot description, xacro)
@@ -12,14 +12,16 @@
   </gazebo>
   <gazebo>
-      <plugin filename="gz-sim-diff-drive-system" name="gz::sim::systems::DiffDrive">
+      <plugin name="gz::sim::systems::DiffDrive" filename="gz-sim-diff-drive-system">
           <left_joint>left_wheel_joint</left_joint>
           <right_joint>right_wheel_joint</right_joint>
           <wheel_separation>0.425</wheel_separation>
           <wheel_radius>0.1</wheel_radius>
-          <topic>/cmd_vel</topic>
+          <odom_publish_frequency>50</odom_publish_frequency>
+          <topic>/model/my_car/cmd_vel</topic>        <!-- Must be Same as Gazebo bridge topic name-->
           <frame_id>odom</frame_id>
           <child_frame_id>base_footprint</child_frame_id>
           <publish_tf>true</publish_tf>
           <odom_topic>/odom</odom_topic>
+          <always_on>true</always_on>
       </plugin>
   </gazebo>

File: src/mobile_robot_description/urdf/my_car.urdf.xacro (robot description, xacro)
@@ -3,6 +3,6 @@
     <xacro:include filename = "common_properties.xacro"/>
     <xacro:include filename = "mobile_base.xacro"/>
+    <xacro:include filename = "lidar.xacro"/>
     <xacro:include filename = "camera_sensor.xacro"/>
-    <xacro:include filename = "lidar.xacro"/>
     <xacro:include filename = "mobile_base_gazebo.xacro"/>
 </robot>
